Commit message: Change to add parameters

File: models/xacro_files/rm2_body.xacro (robot description, xacro)
@@ -2,5 +2,5 @@
 <robot name="body" xmlns:xacro="http://wiki.ros.org/xacro">
 <xacro:macro name="body" params="sufix ">
-  <link name='bodyBase_body_${sufix}'>
+  <link name='bodyBase_${sufix}'>
       <visual>
         <origin rpy="0 0 0" xyz="0 0 0"/>
@@ -22,20 +22,20 @@
     </inertial>
   </link>
-  <link name="AttachableLink_1_body_${sufix}"/>
-  <joint name="AttachableLinkJoint_1_body_${sufix}" type="fixed">
-    <parent link="bodyBase_body_${sufix}"/>
-    <child link="AttachableLink_1_body_${sufix}"/>
+  <link name="AttachableLink_1_${sufix}"/>
+  <joint name="AttachableLinkJoint_1_${sufix}" type="fixed">
+    <parent link="bodyBase_${sufix}"/>
+    <child link="AttachableLink_1_${sufix}"/>
     <origin rpy="0 0 0" xyz="0.0 0 0.085"/>
   </joint>
-  <link name="AttachableLink_2_body_${sufix}"/>
-  <joint name="AttachableLinkJoint_2_body_${sufix}" type="fixed">
-    <parent link="bodyBase_body_${sufix}"/>
-    <child link="AttachableLink_2_body_${sufix}"/>
+  <link name="AttachableLink_2_${sufix}"/>
+  <joint name="AttachableLinkJoint_2_${sufix}" type="fixed">
+    <parent link="bodyBase_${sufix}"/>
+    <child link="AttachableLink_2_${sufix}"/>
     <origin rpy="-2.0944 0 0" xyz="0.0 0.0736 -0.0425"/>
   </joint>
-  <link name="AttachableLink_3_body_${sufix}"/>
-  <joint name="AttachableLinkJoint_3_body_${sufix}" type="fixed">
-    <parent link="bodyBase_body_${sufix}"/>
-    <child link="AttachableLink_3_body_${sufix}"/>
+  <link name="AttachableLink_3_${sufix}"/>
+  <joint name="AttachableLinkJoint_3_${sufix}" type="fixed">
+    <parent link="bodyBase_${sufix}"/>
+    <child link="AttachableLink_3_${sufix}"/>
     <origin rpy="2.0944 0 0" xyz="0.0 -0.0736 -0.0425"/>
   </joint>

File: models/xacro_files/rm2_leg.xacro (robot description, xacro)
@@ -2,5 +2,5 @@
 <robot name= "leg" xmlns:xacro="http://wiki.ros.org/xacro">
   <xacro:macro name="leg" params="sufix ">
-    <link name="legLink_leg_${sufix}">
+    <link name="legLink_${sufix}">
       <visual>
         <origin rpy="0.0 0 0" xyz="0 0 0"/>
@@ -21,5 +21,5 @@
     </link>
     <!-- INCLUDE FRAME MOTOR 1 -->
-    <link name="fm1Link_leg_${sufix}">
+    <link name="fm1Link_${sufix}">
       <visual>
         <origin rpy="0 0 0" xyz="-0.0132 0 -0.01"/> <!--pose relative_to="j_l_fm1">-0.013863 -0.019021 -0.01165 0 0 0</pose-->
@@ -41,7 +41,7 @@
     </link>
     <!-- JOINT LEG - FRAME MOTOR 1 -->
-    <joint name="j_l_fm1_leg_${sufix}" type="fixed">
-      <parent link="legLink_leg_${sufix}"/>
-      <child link="fm1Link_leg_${sufix}"/>
+    <joint name="j_l_fm1_${sufix}" type="fixed">
+      <parent link="legLink_${sufix}"/>
+      <child link="fm1Link_${sufix}"/>
       <axis xyz="0 1 0"/>
       <origin rpy="0 0 0" xyz="0.067490 0 0.009020"/>
@@ -51,5 +51,5 @@
     </joint>
     <!-- INCLUDE FRAME MOTOR 2 -->
-    <link name="fm2Link_leg_${sufix}">
+    <link name="fm2Link_${sufix}">
       <visual>
         <origin rpy="0.0 0 0" xyz="0.0125 0 -0.0134"/>
@@ -73,13 +73,13 @@
     </link>
     <!-- JOINT LEG - FRAME MOTOR 2 -->
-    <joint name="j_l_fm2_leg_${sufix}" type="fixed">
-      <axis xyz="0 1 0"/>
-      <parent link="legLink_leg_${sufix}"/>
-      <child link="fm2Link_leg_${sufix}"/>
+    <joint name="j_l_fm2_${sufix}" type="fixed">
+      <axis xyz="0 1 0"/>
+      <parent link="legLink_${sufix}"/>
+      <child link="fm2Link_${sufix}"/>
       <origin rpy="0 0 0" xyz="-0.057399 0.018994 0.012734"/>
       <!--pose relative_to="legLink">-0.057399 0.018994 0.012734 0 0 0</pose-->
     </joint>
     <!-- INCLUDE FRAME MOTOR 3 -->
-    <link name="fm3Link_leg_${sufix}">
+    <link name="fm3Link_${sufix}">
       <visual>
         <origin rpy="0 0 0" xyz="-0.0132 0 -0.0140"/>
@@ -103,13 +103,13 @@
     </link>
     <!-- JOINT LEG - FRAME MOTOR 3 -->
-    <joint name="j_l_fm3_leg_${sufix}" type="fixed">
-      <axis xyz="0 1 0"/>
-      <parent link="legLink_leg_${sufix}"/>
-      <child link="fm3Link_leg_${sufix}"/>
+    <joint name="j_l_fm3_${sufix}" type="fixed">
+      <axis xyz="0 1 0"/>
+      <parent link="legLink_${sufix}"/>
+      <child link="fm3Link_${sufix}"/>
       <origin rpy="0 0 0" xyz="-0.012 -0.018994 0.012734"/>
       <!--pose relative_to="legLink">-0.012388 -0.019006 0.012734 0 0 0</pose-->
     </joint>
     <!-- INCLUDE FRAME ACTUATOR 1 -->
-    <link name="fa1Link_leg_${sufix}">
+    <link name="fa1Link_${sufix}">
       <visual>
         <origin rpy="0 0 0" xyz="0.01 0 0.03"/>
@@ -133,13 +133,13 @@
     </link>
     <!-- JOINT FRAME MOTOR 1 - FRAME ACTUATOR 1 -->
-    <joint name="j_fm1_fa1_leg_${sufix}" type="fixed">
-      <axis xyz="0 1 0"/>
-      <parent link="fm1Link_leg_${sufix}"/>
-      <child link="fa1Link_leg_${sufix}"/>
+    <joint name="j_fm1_fa1_${sufix}" type="fixed">
+      <axis xyz="0 1 0"/>
+      <parent link="fm1Link_${sufix}"/>
+      <child link="fa1Link_${sufix}"/>
       <origin rpy="0 0 0" xyz="-0.03865 0 -0.03721"/>
       <!--pose relative_to="fm1Link"> -0.028265 0.021 -0.023721 0 0 0 </pose-->
     </joint>
     <!-- INCLUDE FRAME ACTUATOR 2 -->
-    <link name="fa2Link_leg_${sufix}">
+    <link name="fa2Link_${sufix}">
       <visual>
         <origin rpy="0 0 0" xyz="-0.01 0 0.025"/>
@@ -163,13 +163,13 @@
     </link>
     <!-- JOINT FRAME MOTOR 2 - FRAME ACTUATOR 2 -->
-    <joint name="j_fm2_fa2_leg_${sufix}" type="fixed">
-      <axis xyz="0 1 0"/>
-      <parent link="fm2Link_leg_${sufix}"/>
-      <child link="fa2Link_leg_${sufix}"/>
+    <joint name="j_fm2_fa2_${sufix}" type="fixed">
+      <axis xyz="0 1 0"/>
+      <parent link="fm2Link_${sufix}"/>
+      <child link="fa2Link_${sufix}"/>
       <origin rpy="0 0 0" xyz="0.03865 0.000851 -0.03721"/>-
       <!--pose relative_to="fm2Link"> 0.028265 0.000851 -0.023717 0 0 0 </pose-->
     </joint>
   <!-- INCLUDE FRAME ACTUATOR 3 -->
-    <link name="fa3Link_leg_${sufix}">
+    <link name="fa3Link_${sufix}">
       <visual>
         <origin rpy="0 0 0" xyz="0.01 0 0.025"/>
@@ -193,12 +193,12 @@
     </link>
     <!-- JOINT FRAME MOTOR 3 - FRAME ACTUATOR 3 -->
-    <joint name="j_fm3_fa3_leg_${sufix}" type="fixed">
-      <axis xyz="0 1 0"/>
-      <parent link="fm3Link_leg_${sufix}"/>
-      <child link="fa3Link_leg_${sufix}"/>
+    <joint name="j_fm3_fa3_${sufix}" type="fixed">
+      <axis xyz="0 1 0"/>
+      <parent link="fm3Link_${sufix}"/>
+      <child link="fa3Link_${sufix}"/>
       <origin rpy="0 0 0" xyz="-0.038265 -0.000851 -0.03721"/>
       <!--pose relative_to="fm3Link"> -0.028265 -0.000851 -0.023717 0 0 0</pose-->
     </joint>
-  <link name="AttachableLink_1_leg_${sufix}">
+  <link name="AttachableLink_1_${sufix}">
     <!--visual>
       <origin xyz="0 0 0.05" rpy= "0 0 0" />
@@ -208,7 +208,7 @@
     </visual-->
   </link>
-  <joint name="AttachableLinkJoint_1_leg_${sufix}" type="fixed">
-    <parent link="AttachableLink_1_leg_${sufix}"/>
-    <child link="legLink_leg_${sufix}"/>
+  <joint name="AttachableLinkJoint_1_${sufix}" type="fixed">
+    <parent link="AttachableLink_1_${sufix}"/>
+    <child link="legLink_${sufix}"/>
     <origin rpy="0 0 0" xyz="-0.005 0 0"/>
   </joint>
