Commit message: Update repo

File: models/actual_model/actual_model.xacro (robot description, xacro)
@@ -1,5 +1,4 @@
 <robot xmlns:xacro="http://wiki.ros.org/xacro" name="test">
   <xacro:include filename="$(find attachable_pkg)/models/xacro_files/import_path.xacro"/>
-  <xacro:body sufix="body_1">
-  </xacro:body>
-  <xacro:leg sufix="leg_1"/><joint name="AttachableJoint_body_1_AttachableLink_1_body_1_leg_1_AttachableLink_1_leg_1" type="fixed"><parent link="AttachableLink_1_body_1"/><child link="AttachableLink_1_leg_1"/><origin rpy="0 0 0" xyz="0 0 0"/></joint></robot>
+  <xacro:body sufix="body_1"/>
+</robot>

File: models/actual_model/template.xacro (robot description, xacro)
@@ -1,5 +1,4 @@
 <robot xmlns:xacro="http://wiki.ros.org/xacro" name="test">
   <xacro:include filename="$(find attachable_pkg)/models/xacro_files/import_path.xacro" />
-  <xacro:body sufix="body_1">
-  </xacro:body>
-  </robot>
+  <xacro:body sufix="body_1"/>
+</robot>

File: models/urdf/rm2_body.urdf (robot description, URDF)
Before this commit: robot body, 0 links, 0 joints
Links:
- added link AttachableLink_1_1
- added link AttachableLink_2_1
- added link AttachableLink_3_1
- added link bodyBase_1, mass 1.8; collision mesh filename=package://rm2_simulation/models/rm2_body/meshes/body_collis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; visual mesh filename=package://rm2_simulation/models/rm2_body/meshes/b_simple.dae
Joints:
- added joint AttachableLinkJoint_1_1: type fixed, parent bodyBase_1, child AttachableLink_1_1, origin xyz=0.0 0 0.085 rpy=0 0 0
- added joint AttachableLinkJoint_2_1: type fixed, parent bodyBase_1, child AttachableLink_2_1, origin xyz=0.0 0.0736 -0.0425 rpy=-2.0944 0 0
- added joint AttachableLinkJoint_3_1: type fixed, parent bodyBase_1, child AttachableLink_3_1, origin xyz=0.0 -0.0736 -0.0425 rpy=2.0944 0 0
