Commit message: TEST 1

File: models/actual_model/actual_model.urdf (robot description, URDF)
Before this commit: robot test, 4 links, 3 joints
Links:
- removed link AttachableLink_1_body_1
- removed link AttachableLink_2_body_1
- removed link AttachableLink_3_body_1
- removed link bodyBase_body_1
- added link AttachableLink_1_rm2_1
- added link AttachableLink_2_rm2_1
- added link base_link_rm2_1
- added link d_435_camera_rm2_1
- added link l1::fLink_rm2_1
- added link l1::lLink_rm2_1
- added link l1::mLink_rm2_1
- added link l2::fLink_rm2_1
- added link l2::lLink_rm2_1
- added link l2::mLink_rm2_1
- added link l3::fLink_rm2_1
- added link l3::lLink_rm2_1
- added link l3::mLink_rm2_1
- added link lidar_rm2_1
- added link sa1::aLink_rm2_1
- added link sa1::sbLink_rm2_1
- added link sa2::aLink_rm2_1
- added link sa2::sbLink_rm2_1
- added link sa3::aLink_rm2_1
- added link sa3::sbLink_rm2_1
- added link wa2::aLink_rm2_1
- added link wa2::wbLink_rm2_1
- added link wa3::aLink_rm2_1
- added link wa3::wbLink_rm2_1
Joints:
- removed joint AttachableLinkJoint_1_body_1
- removed joint AttachableLinkJoint_2_body_1
- removed joint AttachableLinkJoint_3_body_1
- added joint AttachableLinkJoint_1_rm2_1: type fixed, parent base_link_rm2_1, child AttachableLink_1_rm2_1, origin xyz=0.0 -0.0736 -0.0425 rpy=2.0944 0 0
- added joint AttachableLinkJoint_2_rm2_1: type fixed, parent base_link_rm2_1, child AttachableLink_2_rm2_1, origin xyz=0.0 -0.0736 -0.0425 rpy=2.0944 0 0
- added joint j_b_l1: type fixed, parent base_link_rm2_1, child l1::lLink_rm2_1, origin xyz=0.0035 0.024 0.0473 rpy=0 0 0
- added joint j_b_l2: type fixed, parent base_link_rm2_1, child l2::lLink_rm2_1, origin xyz=0.083 0.065 -0.0375 rpy=-2.0944 0 0
- added joint j_b_l3: type fixed, parent base_link_rm2_1, child l3::lLink_rm2_1, origin xyz=0.083 -0.065 -0.0375 rpy=2.0944 0 0
- added joint j_l1_sa1: type fixed, parent l1::fLink_rm2_1, child sa1::aLink_rm2_1, origin xyz=0.0035 0.024 0.0473 rpy=0 0 0
- added joint j_l2_sa2: type fixed, parent l2::fLink_rm2_1, child sa2::aLink_rm2_1, origin xyz=0.0035 0.024 0.0473 rpy=0 0 0
- added joint j_l2_wa2: type fixed, parent l2::fLink_rm2_1, child wa2::aLink_rm2_1, origin xyz=0.0035 0.024 0.0473 rpy=0 0 0
- added joint j_l3_sa3: type fixed, parent l3::fLink_rm2_1, child sa3::aLink_rm2_1, origin xyz=0.0035 0.024 0.0473 rpy=0 0 0
- added joint j_l3_wa3: type fixed, parent l3::fLink_rm2_1, child wa3::aLink_rm2_1, origin xyz=0.0035 0.024 0.0473 rpy=0 0 0
- added joint j_lidar_b: type fixed, parent base_link_rm2_1, child lidar_rm2_1, origin xyz=0.0 0 0.25 rpy=0 0 0
- added joint j_rgbd_b: type fixed, parent base_link_rm2_1, child d_435_camera_rm2_1, origin xyz=0.090 0 0.038911 rpy=0 0 0
- added joint l1::j_l_m: type fixed, parent l1::lLink_rm2_1, child l1::mLink_rm2_1, origin xyz=0 0 0 rpy=0 0 0
- added joint l1::j_m_f: type fixed, parent l1::mLink_rm2_1, child l1::fLink_rm2_1, origin xyz=0.0153 0.019 0.0135 rpy=0 0 0
- added joint l2::j_l_m: type fixed, parent l2::lLink_rm2_1, child l2::mLink_rm2_1, origin xyz=0 0 0 rpy=0 0 0
- added joint l2::j_m_f: type fixed, parent l2::mLink_rm2_1, child l2::fLink_rm2_1, origin xyz=0.0153 0.019 0.0135 rpy=0 0 0
- added joint l3::j_l_m: type fixed, parent l3::lLink_rm2_1, child l3::mLink_rm2_1, origin xyz=0 0 0 rpy=0 0 0
- added joint l3::j_m_f: type fixed, parent l3::mLink_rm2_1, child l3::fLink_rm2_1, origin xyz=0.0153 0.019 0.0135 rpy=0 0 0
- added joint sa1::j_a_sb: type fixed, parent sa1::aLink_rm2_1, child sa1::sbLink_rm2_1, origin xyz=0 0 0 rpy=0 0 0
- added joint sa2::j_a_sb: type fixed, parent sa2::aLink_rm2_1, child sa2::sbLink_rm2_1, origin xyz=0 0 0 rpy=0 0 0
- added joint sa3::j_a_sb: type fixed, parent sa3::aLink_rm2_1, child sa3::sbLink_rm2_1, origin xyz=0 0 0 rpy=0 0 0
- added joint wa2::j_a_wb: type fixed, parent wa2::aLink_rm2_1, child wa2::wbLink_rm2_1, origin xyz=0 0 0.0025 rpy=0 1.5708 0
- added joint wa3::j_a_wb: type fixed, parent wa3::aLink_rm2_1, child wa3::wbLink_rm2_1, origin xyz=0 0 0.0025 rpy=0 1.5708 0

File: models/actual_model/actual_model.xacro (robot description, xacro)
@@ -1,4 +1,5 @@
 <robot xmlns:xacro="http://wiki.ros.org/xacro" name="test">
-  <xacro:include filename="$(find attachable_pkg)/models/xacro_files/import_path.xacro"/>
-  <xacro:body sufix="body_1"/>
+  <xacro:include filename="$(find attachable_pkg)/models/xacro_files/import_path.xacro" />
+  <!--xacro:body sufix="body_1"/-->
+  <xacro:rm2_p sufix="rm2_1"/>
 </robot>

File: models/actual_model/template.xacro (robot description, xacro)
@@ -1,4 +1,5 @@
 <robot xmlns:xacro="http://wiki.ros.org/xacro" name="test">
   <xacro:include filename="$(find attachable_pkg)/models/xacro_files/import_path.xacro" />
-  <xacro:body sufix="body_1"/>
+  <!--xacro:body sufix="body_1"/-->
+  <xacro:rm2_p sufix="rm2_1"/>
 </robot>

File: models/other/myfirst.xacro (robot description, xacro)
@@ -1,18 +1,4 @@
 <robot xmlns:xacro="http://wiki.ros.org/xacro" name="test">
-  <xacro:include filename="import_path.xacro"/>
-  <!--xacro:include filename="rm2_leg.xacro" />
-  <xacro:include filename="rm2_body.xacro" /-->
-  <!--xacro:macro name="blue_shape">
-      <link name="base1">
-      <visual>
-        <geometry>
-          <cylinder length="0.6" radius="0.2"/>
-        </geometry>
-      </visual>
-    </link>
-  </xacro:macro
-  AttachableLink_leg1
-  legLink_leg1
-  -->
+  <xacro:include filename="$(find attachable_pkg)/models/xacro_files/import_path.xacro" />
   <xacro:body sufix="1">
   </xacro:body>

File: models/xacro_files/import_path.xacro (robot description, xacro)
@@ -3,5 +3,11 @@
   <!--xacro:include filename="../models/rm2_body.xacro" />
   <xacro:include filename="../models/rm2_leg.xacro" /-->
-  <xacro:include filename="$(find attachable_pkg)/models/xacro_files/rm2_body.xacro"/>
-  <xacro:include filename="$(find attachable_pkg)/models/xacro_files/rm2_leg.xacro" />
+  <xacro:include filename="$(find attachable_pkg)/models/xacro_files/rm2_body_p.xacro"/>
+  <xacro:include filename="$(find attachable_pkg)/models/xacro_files/rm2_body_c_1.xacro"/>
+  <xacro:include filename="$(find attachable_pkg)/models/xacro_files/rm2_body_c_2.xacro"/>
+  <xacro:include filename="$(find attachable_pkg)/models/xacro_files/rm2_body_c_3.xacro"/>
+  <xacro:include filename="$(find attachable_pkg)/models/xacro_files/rm2_leg_c_1.xacro" />
+  <xacro:include filename="$(find attachable_pkg)/models/xacro_files/rm2_p.xacro" />
+  <xacro:include filename="$(find attachable_pkg)/models/xacro_files/rm2_c_1.xacro" />
+  <xacro:include filename="$(find attachable_pkg)/models/xacro_files/rm2_c_2.xacro" />
 </robot>

File: models/xacro_files/rm2_body_p.xacro (robot description, xacro)
@@ -1,5 +1,5 @@
 <?xml version="1.0"?>
-<robot name="body" xmlns:xacro="http://wiki.ros.org/xacro">
-<xacro:macro name="body" params="sufix ">
+<robot name="body_p" xmlns:xacro="http://wiki.ros.org/xacro">
+<xacro:macro name="body_p" params="sufix ">
   <link name='bodyBase_${sufix}'>
       <visual>

File: models/xacro_files/rm2_leg_c_1.xacro (robot description, xacro)
@@ -1,5 +1,5 @@
 <?xml version="1.0"?>
-<robot name= "leg" xmlns:xacro="http://wiki.ros.org/xacro">
-  <xacro:macro name="leg" params="sufix ">
+<robot name= "leg_c_1" xmlns:xacro="http://wiki.ros.org/xacro">
+  <xacro:macro name="leg_c_1" params="sufix ">
     <link name="legLink_${sufix}">
       <visual>
